File: Hardware/V4/ESP32-Cam-Pico-V4.brd (EAGLE design)
At the start: 28.6 x 57.1 mm, 45 parts, among them IC1 ESP32-CAM, IC2 MCP170333MB, J4 JST_ZH_2PIN, U1 HX4002

Commit message: Commit post first flight
Parts:
- added C13: 4.7uF, SparkFun-Capacitors:0402
- moved J4 0.32 mm to (21.6, 48.9)
- moved C11 0.32 mm to (23.8, 50.2)
- moved IC2 0.13 mm to (17.6, 44.5)
Connections:
- net GND: now also C13.2
- net S+: now also C13.1
Routing:
- net GND: track 25.8 -> 39.6 mm
- net S+: track 146.5 -> 149.2 mm
